Commit message: renamed base_link + missing dep

File: urdf/ovis_arm.xacro (robot description, xacro)
@@ -5,9 +5,9 @@
       <joint name="${arm_id}_joint_${connected_to}" type="fixed">
         <parent link="${connected_to}"/>
-        <child link="${arm_id}_link0"/>
+        <child link="${arm_id}_base_link"/>
         <origin rpy="${rpy}" xyz="${xyz}"/>
       </joint>
     </xacro:unless>
-    <link name="${arm_id}_link0">
+    <link name="${arm_id}_base_link">
       <visual>
         <geometry>
@@ -45,5 +45,5 @@
     <joint name="${arm_id}_joint1" type="revolute">
       <origin xyz="0 0 0.051" rpy="0 0 0"/>
-      <parent link="${arm_id}_link0"/>
+      <parent link="${arm_id}_base_link"/>
       <child link="${arm_id}_link1"/>
       <dynamics damping="0.1"/>

Commit message: description refactor using ros_industrial guidelines

File: urdf/ovis_arm.xacro (robot description, xacro)
@@ -151,11 +151,11 @@
       <limit effort="10000.0" lower="${-2*pi}" upper="${2*pi}" velocity="0.57"/>
     </joint>
-    <link name="${arm_id}_link7">
+    <link name="${arm_id}_tool0">
     </link>
-    <joint name="moveit_handle" type="fixed">
-    <parent link="${arm_id}_link6"/>
-    <child link="${arm_id}_link7"/>
-    <origin xyz="0 0 -0.26995" rpy="0 ${pi} ${pi/2}"/>
-  </joint>
+    <joint name="${arm_id}_link6-tool0" type="fixed">
+      <parent link="${arm_id}_link6"/>
+      <child link="${arm_id}_tool0"/>
+      <origin xyz="0 0 -0.09215" rpy="0 ${pi} ${pi/2}"/>
+    </joint>
   </xacro:macro>
 </robot>

File: urdf/ovis_w_gripper.xacro (robot description, xacro)
@@ -8,7 +8,14 @@
   <!-- attach robotiq gripper to ovis flange -->
   <joint name="gripper_base" type="fixed">
-    <parent link="ovis_link6"/>
+    <parent link="ovis_tool0"/>
     <child link="robotiq_arg2f_base_link"/>
-    <origin xyz="0 0 -0.09215" rpy="0 ${pi} ${pi/2}"/>
+    <origin xyz="0 0 0" rpy="0 0 0"/>
+  </joint>
+  <!-- define a virtual pivot point for moveit -->
+  <link name="virtual_pivot"/>
+  <joint name="moveit_handle" type="fixed">
+    <parent link="robotiq_arg2f_base_link"/>
+    <child link="virtual_pivot"/>
+    <origin xyz="0 0 0.1778" rpy="0 0 0"/>
   </joint>
 </robot>
