Commit message: added simulated camera to urdf.

File: urdf/ovis.xacro (robot description, xacro)
@@ -3,4 +3,5 @@
 <root xmlns:xi="http://www.w3.org/2001/XInclude"
     xmlns:xacro="http://www.ros.org/wiki/xacro">
+    <xacro:include filename="$(find ovis_description)/urdf/ovis.gazebo" />
     <xacro:include filename="$(find ovis_description)/urdf/kinova_common.xacro" />
     <xacro:property name="link_base_mesh" value="ovis_base" />
@@ -83,4 +84,9 @@
     <xacro:property name="joint_end_effector_origin_xyz" value="0 0 0.1778" />
     <xacro:property name="joint_end_effector_origin_rpy" value="0 0 0" />
+    <xacro:property name="joint_camera" value="camera" />
+    <xacro:property name="joint_camera_type" value="fixed" />
+    <xacro:property name="joint_camera_axis_xyz" value="0 0 0" />
+    <xacro:property name="joint_camera_origin_xyz" value="0 0.091842 -0.0732" />
+    <xacro:property name="joint_camera_origin_rpy" value="0 ${pi} ${pi/2}" />
     <xacro:macro name="ovis" params="base_parent prefix:=ovis">
         <xacro:kinova_armlink link_name="${prefix}_link_base" link_mesh="${link_base_mesh}" link_origin_rpy="${link_base_origin_rpy}"/>
@@ -102,4 +108,7 @@
         <xacro:kinova_virtual_link link_name="${prefix}_end_effector"/>
         <xacro:kinova_virtual_joint joint_name="${prefix}_joint_end_effector" type="${joint_end_effector_type}" parent="${prefix}_link_tool0" child="${prefix}_end_effector" joint_axis_xyz="${joint_end_effector_axis_xyz}" joint_origin_xyz="${joint_end_effector_origin_xyz}" joint_origin_rpy="${joint_end_effector_origin_rpy}" joint_lower_limit="0" joint_upper_limit="0"/>
+        <!-- Camera -->
+        <xacro:kinova_virtual_link link_name="${prefix}_camera"/>
+        <xacro:kinova_virtual_joint joint_name="${prefix}_camera" type="${joint_camera_type}" parent="${prefix}_link_6" child="${prefix}_camera" joint_axis_xyz="${joint_camera_axis_xyz}" joint_origin_xyz="${joint_camera_origin_xyz}" joint_origin_rpy="${joint_camera_origin_rpy}" joint_lower_limit="0" joint_upper_limit="0"/>
     </xacro:macro>
 </root>

Commit message: added launch for display in gazebo.

File: urdf/ovis.xacro (robot description, xacro)
@@ -86,7 +86,20 @@
     <xacro:property name="joint_camera" value="camera" />
     <xacro:property name="joint_camera_type" value="fixed" />
-    <xacro:property name="joint_camera_axis_xyz" value="0 0 0" />
-    <xacro:property name="joint_camera_origin_xyz" value="0 0.091842 -0.0732" />
+    <xacro:property name="joint_camera_axis_xyz" value="0 0 1" />
+    <!-- <xacro:property name="joint_camera_origin_xyz" value="0 0.091842 -0.0732" /> -->
+    <xacro:property name="joint_camera_origin_xyz" value="0 0.091842 -0.125" />
     <xacro:property name="joint_camera_origin_rpy" value="0 ${pi} ${pi/2}" />
+    <link name="ovis_camera">
+        <inertial>
+            <mass value=".1"/>
+            <origin rpy="0 0 0" xyz="0 0 0"/>
+            <inertia ixx="0" ixy="0.0" ixz="0.0" iyy="0" iyz="0.0" izz="0" />
+        </inertial>
+        <visual>
+            <geometry>
+                <box size=".01 .01 .01"/>
+            </geometry>
+        </visual>
+    </link>
     <xacro:macro name="ovis" params="base_parent prefix:=ovis">
         <xacro:kinova_armlink link_name="${prefix}_link_base" link_mesh="${link_base_mesh}" link_origin_rpy="${link_base_origin_rpy}"/>
@@ -109,6 +122,7 @@
         <xacro:kinova_virtual_joint joint_name="${prefix}_joint_end_effector" type="${joint_end_effector_type}" parent="${prefix}_link_tool0" child="${prefix}_end_effector" joint_axis_xyz="${joint_end_effector_axis_xyz}" joint_origin_xyz="${joint_end_effector_origin_xyz}" joint_origin_rpy="${joint_end_effector_origin_rpy}" joint_lower_limit="0" joint_upper_limit="0"/>
         <!-- Camera -->
-        <xacro:kinova_virtual_link link_name="${prefix}_camera"/>
+        <!-- <xacro:kinova_virtual_link link_name="${prefix}_camera"/> -->
         <xacro:kinova_virtual_joint joint_name="${prefix}_camera" type="${joint_camera_type}" parent="${prefix}_link_6" child="${prefix}_camera" joint_axis_xyz="${joint_camera_axis_xyz}" joint_origin_xyz="${joint_camera_origin_xyz}" joint_origin_rpy="${joint_camera_origin_rpy}" joint_lower_limit="0" joint_upper_limit="0"/>
+        <!-- camera link -->
     </xacro:macro>
 </root>

Commit message: minimal gazebo simulation

File: urdf/ovis.xacro (robot description, xacro)
@@ -87,7 +87,6 @@
     <xacro:property name="joint_camera_type" value="fixed" />
     <xacro:property name="joint_camera_axis_xyz" value="0 0 1" />
-    <!-- <xacro:property name="joint_camera_origin_xyz" value="0 0.091842 -0.0732" /> -->
-    <xacro:property name="joint_camera_origin_xyz" value="0 0.091842 -0.125" />
-    <xacro:property name="joint_camera_origin_rpy" value="0 ${pi} ${pi/2}" />
+    <xacro:property name="joint_camera_origin_xyz" value="0 0.091842 -0.0732" />
+    <xacro:property name="joint_camera_origin_rpy" value="0 ${pi/2} ${pi/2}" />
     <link name="ovis_camera">
         <inertial>

Commit message: urdf clean up + added colors to gazebo sim

File: urdf/ovis.xacro (robot description, xacro)
@@ -89,4 +89,5 @@
     <xacro:property name="joint_camera_origin_xyz" value="0 0.091842 -0.0732" />
     <xacro:property name="joint_camera_origin_rpy" value="0 ${pi/2} ${pi/2}" />
+    <!-- camera link -->
     <link name="ovis_camera">
         <inertial>
@@ -95,9 +96,9 @@
             <inertia ixx="0" ixy="0.0" ixz="0.0" iyy="0" iyz="0.0" izz="0" />
         </inertial>
-        <visual>
+        <!-- <visual>
             <geometry>
                 <box size=".01 .01 .01"/>
             </geometry>
-        </visual>
+        </visual> -->
     </link>
     <xacro:macro name="ovis" params="base_parent prefix:=ovis">
@@ -121,7 +122,5 @@
         <xacro:kinova_virtual_joint joint_name="${prefix}_joint_end_effector" type="${joint_end_effector_type}" parent="${prefix}_link_tool0" child="${prefix}_end_effector" joint_axis_xyz="${joint_end_effector_axis_xyz}" joint_origin_xyz="${joint_end_effector_origin_xyz}" joint_origin_rpy="${joint_end_effector_origin_rpy}" joint_lower_limit="0" joint_upper_limit="0"/>
         <!-- Camera -->
-        <!-- <xacro:kinova_virtual_link link_name="${prefix}_camera"/> -->
         <xacro:kinova_virtual_joint joint_name="${prefix}_camera" type="${joint_camera_type}" parent="${prefix}_link_6" child="${prefix}_camera" joint_axis_xyz="${joint_camera_axis_xyz}" joint_origin_xyz="${joint_camera_origin_xyz}" joint_origin_rpy="${joint_camera_origin_rpy}" joint_lower_limit="0" joint_upper_limit="0"/>
-        <!-- camera link -->
     </xacro:macro>
 </root>

Commit message: Updated inertial properties to better reflect the reality

File: urdf/ovis.xacro (robot description, xacro)
@@ -24,4 +24,5 @@
     <xacro:property name="joint_1_axis_xyz" value="0 0 1" />
     <xacro:property name="joint_1_origin_xyz" value="0 0 0.051" />
+    <!-- New Z offset to be 0.06885 -->
     <xacro:property name="joint_1_origin_rpy" value="0 0 0" />
     <xacro:property name="joint_1_lower_limit" value="${-4*pi}" />

File: urdf/ovis_inertial.xacro (robot description, xacro)
@@ -17,7 +17,7 @@
         <xacro:if value="${link_name == 'ovis_link_base'}">
             <inertial>
-                <mass value="16.111" />
-                <origin xyz="-0.00002529 0.00000008 -0.06049447" rpy="0 0 0"/>
-                <inertia ixx="0.385006414" ixy="0.0000696244868" ixz="-0.000181517937" iyy="0.624959190" iyz="0.000000162897534" izz="0.798949961"/>
+                <mass value="1.53" />
+                <origin xyz="0 0 0.04385330" rpy="0 0 0"/>
+                <inertia ixx="0.00320907"  ixy="2e-008"  ixz="2e-008" iyy="0.00321098" iyz="-6e-007" izz="0.0056695" />
             </inertial>
         </xacro:if>
@@ -25,7 +25,7 @@
         <xacro:if value="${link_name == 'ovis_link_1'}">
             <inertial>
-                <mass value="0.7477"/>
-                <origin xyz="0 -0.002 -0.0605" rpy="0 0 0"/>
-                <inertia ixx="0.385006414" ixy="0.0000696244868" ixz="-0.000181517937" iyy="0.624959190" iyz="0.000000162897534" izz="0.798949961"/>
+                <mass value="1.2" />
+                <origin xyz="0 -0.0111 0.055" rpy="0 0 0"/>
+                <inertia ixx="0.00248772"  ixy="-1.6e-007"  ixz="2.2e-007" iyy="0.0027245" iyz="-0.00031134" izz="0.00126329" />
             </inertial>
         </xacro:if>
@@ -33,15 +33,15 @@
         <xacro:if value="${link_name == 'ovis_link_2'}">
             <inertial>
-                <mass value="0.7477"/>
-                <origin xyz="0 -0.002 -0.0605" rpy="0 0 0"/>
-                <inertia ixx="0.385006414" ixy="0.0000696244868" ixz="-0.000181517937" iyy="0.624959190" iyz="0.000000162897534" izz="0.798949961"/>
-            </inertial>
+                <mass value="1.3" />
+                <origin xyz="0 0.17553971 -0.00935895" rpy="0 0 0"/>
+                <inertia ixx="0.03068681"  ixy="1.76e-006"  ixz="1e-007" iyy="0.00109408" iyz="0.00018345" izz="0.03103519" />
+           </inertial>
         </xacro:if>
         <!-- Link 3 -->
         <xacro:if value="${link_name == 'ovis_link_3'}">
             <inertial>
-                <mass value="0.7477"/>
-                <origin xyz="0 -0.002 -0.0605" rpy="0 0 0"/>
-                <inertia ixx="0.385006414" ixy="0.0000696244868" ixz="-0.000181517937" iyy="0.624959190" iyz="0.000000162897534" izz="0.798949961"/>
+                <mass value="0.592" />
+                <origin xyz="0.03828435 0.01104986 0.00979839" rpy="0 0 0"/>
+                <inertia ixx="0.00049443"  ixy="0.00033167"  ixz="-0.00021435" iyy="0.00147579" iyz="-6.259e-005" izz="0.0016474" />
             </inertial>
         </xacro:if>
@@ -49,7 +49,7 @@
         <xacro:if value="${link_name == 'ovis_link_4'}">
             <inertial>
-                <mass value="0.7477"/>
-                <origin xyz="0 -0.002 -0.0605" rpy="0 0 0"/>
-                <inertia ixx="0.385006414" ixy="0.0000696244868" ixz="-0.000181517937" iyy="0.624959190" iyz="0.000000162897534" izz="0.798949961"/>
+                <mass value="0.652" />
+                <origin xyz="0.00011113 0.12506366 0.00482529" rpy="0 0 0"/>
+                <inertia ixx="0.00685564"  ixy="-4.5e-006"  ixz="-4.1e-007" iyy="0.00052903" iyz="0.00038138" izz="0.00686163" />
             </inertial>
         </xacro:if>
@@ -57,7 +57,7 @@
         <xacro:if value="${link_name == 'ovis_link_5'}">
             <inertial>
-                <mass value="0.7477"/>
-                <origin xyz="0 -0.002 -0.0605" rpy="0 0 0"/>
-                <inertia ixx="0.385006414" ixy="0.0000696244868" ixz="-0.000181517937" iyy="0.624959190" iyz="0.000000162897534" izz="0.798949961"/>
+                <mass value="0.41555" />
+                <origin xyz="0.0 0.03086454 -0.00810577" rpy="0 0 0"/>
+                <inertia ixx="0.00055858"  ixy="-4.3e-007"  ixz="-2.8e-007" iyy="0.00020049" iyz="9.39e-005" izz="0.00057545" />
             </inertial>
         </xacro:if>
@@ -65,7 +65,7 @@
         <xacro:if value="${link_name == 'ovis_link_6'}">
             <inertial>
-                <mass value="0.7477"/>
-                <origin xyz="0 -0.002 -0.0605" rpy="0 0 0"/>
-                <inertia ixx="0.385006414" ixy="0.0000696244868" ixz="-0.000181517937" iyy="0.624959190" iyz="0.000000162897534" izz="0.798949961"/>
+                <mass value="0.6448" />
+                <origin xyz="-0.00120093 0.06932019 -0.00169931" rpy="0 0 0"/>
+                <inertia ixx="0.00326124"  ixy="-1.39e-005"  ixz="-1.38e-006" iyy="0.00125679" iyz="1.69e-005" izz="0.00393291" />
             </inertial>
         </xacro:if>
