Commit message: changed root link name

File: urdf/ovis_standalone.xacro (robot description, xacro)
@@ -13,6 +13,6 @@
     <origin xyz="0 0 0" rpy="0 0 0"/>
   </joint>
-  <link name="root"/>
-  <xacro:property name="robot_root" value="root" />
+  <link name="ovis_root"/>
+  <xacro:property name="robot_root" value="ovis_root" />
   <xacro:ovis base_parent="${robot_root}"/>
 </robot>

Commit message: added joint to world link for gazebo sim

File: urdf/ovis_standalone.xacro (robot description, xacro)
@@ -1,5 +1,17 @@
 <?xml version="1.0"?>
 <!-- OVIS 6DOF spherical wrist robotic arm -->
-<robot xmlns:xacro="http://www.ros.org/wiki/xacro" name="ovis">
+<robot xmlns:xi="http://www.w3.org/2001/XInclude"
+  xmlns:gazebo="http://playerstage.sourceforge.net/gazebo/xmlschema/#gz"
+  xmlns:model="http://playerstage.sourceforge.net/gazebo/xmlschema/#model"
+  xmlns:sensor="http://playerstage.sourceforge.net/gazebo/xmlschema/#sensor"
+  xmlns:body="http://playerstage.sourceforge.net/gazebo/xmlschema/#body"
+  xmlns:geom="http://playerstage.sourceforge.net/gazebo/xmlschema/#geom"
+  xmlns:joint="http://playerstage.sourceforge.net/gazebo/xmlschema/#joint"
+  xmlns:controller="http://playerstage.sourceforge.net/gazebo/xmlschema/#controller"
+  xmlns:interface="http://playerstage.sourceforge.net/gazebo/xmlschema/#interface"
+  xmlns:rendering="http://playerstage.sourceforge.net/gazebo/xmlschema/#rendering"
+  xmlns:renderable="http://playerstage.sourceforge.net/gazebo/xmlschema/#renderable"
+  xmlns:physics="http://playerstage.sourceforge.net/gazebo/xmlschema/#physics"
+  xmlns:xacro="http://www.ros.org/wiki/xacro" name="ovis">
   <!-- Include ovis robotic arm -->
   <xacro:include filename="$(find ovis_description)/urdf/ovis.xacro"/>
@@ -16,3 +28,10 @@
   <xacro:property name="robot_root" value="ovis_root" />
   <xacro:ovis base_parent="${robot_root}"/>
+  <!-- for gazebo -->
+  <link name="world"/>
+  <joint name="connect_root_and_world" type="fixed">
+    <child link="ovis_root" />
+    <parent link="world" />
+    <origin xyz="0 0 0" rpy="0 0 0" />
+  </joint>
 </robot>

Commit message: Removed the world static link to allow integration with markhor

File: urdf/ovis_standalone.xacro (robot description, xacro)
@@ -28,10 +28,3 @@
   <xacro:property name="robot_root" value="ovis_root" />
   <xacro:ovis base_parent="${robot_root}"/>
-  <!-- for gazebo -->
-  <link name="world"/>
-  <joint name="connect_root_and_world" type="fixed">
-    <child link="ovis_root" />
-    <parent link="world" />
-    <origin xyz="0 0 0" rpy="0 0 0" />
-  </joint>
 </robot>
