Commit message: Changed ovis_joint for arm_joint

File: urdf/generated_gazebo.urdf (robot description, URDF)
Before this commit: robot ovis, 12 links, 11 joints
Joints:
- removed joint ovis_joint_1
- removed joint ovis_joint_2
- removed joint ovis_joint_3
- removed joint ovis_joint_4
- removed joint ovis_joint_5
- removed joint ovis_joint_6
- added joint arm_joint_1: type continuous, parent ovis_link_base, child ovis_link_1, origin xyz=0 0 0.051 rpy=0 0 0, axis 0 0 1, limit lower=-12.5663706144 upper=12.5663706144 effort=40 velocity=0.628318530718
- added joint arm_joint_2: type revolute, parent ovis_link_1, child ovis_link_2, origin xyz=0 0 0.0889 rpy=1.57079632679 0 0, axis 0 0 1, limit lower=-1.57079632679 upper=1.57079632679 effort=80 velocity=0.628318530718
- added joint arm_joint_3: type revolute, parent ovis_link_2, child ovis_link_3, origin xyz=0 0.465 0 rpy=0 0 1.57079632679, axis 0 0 1, limit lower=-1.57079632679 upper=1.57079632679 effort=40 velocity=0.628318530718
- added joint arm_joint_4: type continuous, parent ovis_link_3, child ovis_link_4, origin xyz=0.0889 0.047625 0 rpy=0 0 0, axis 0 1 0, limit lower=-12.5663706144 upper=12.5663706144 effort=20 velocity=0.837758040957
- added joint arm_joint_5: type revolute, parent ovis_link_4, child ovis_link_5, origin xyz=0 0.265 0 rpy=0 0 0, axis 0 0 1, limit lower=-1.57079632679 upper=1.57079632679 effort=20 velocity=0.837758040957
- added joint arm_joint_6: type continuous, parent ovis_link_5, child ovis_link_6, origin xyz=0 0.0762 0 rpy=1.57079632679 1.57079632679 0, axis 0 0 1, limit lower=-6.28318530718 upper=6.28318530718 effort=20 velocity=0.837758040957
